Commit message: Added depth sensor to cameras in simulation and updated rviz configuration

File: src/velmwheel/sim/velmwheel_gazebo/velmwheel_gazebo/urdf/camera.urdf.xacro (robot description, xacro)
@@ -14,12 +14,9 @@
 	<xacro:macro name="camera" params="name">
 		<gazebo reference="${name}_color_frame">
-		    <!-- <material>Gazebo/Gray</material> -->
 		    <sensor name="${name}/color" type="camera">
 			    <pose> 0 0 0 0 0 0 </pose>
-			    <visualize>false</visualize>
 			    <update_rate>30</update_rate>
 			    <camera>
 		    	    <horizontal_fov>1.211</horizontal_fov>
-		    	    <vertical_fov>0.742</vertical_fov>
 				    <image>
 				        <format>R8G8B8</format>
@@ -32,6 +29,35 @@
 				    </clip>
 			    </camera>
-			    <plugin name="${name}_controller" filename="libgazebo_ros_camera.so">
+			    <plugin name="${name}_color_controller" filename="libgazebo_ros_camera.so">
 				    <frame_name>${name}_color_optical_frame</frame_name>
+			    </plugin>
+			</sensor>
+		</gazebo>
+		<gazebo reference="${name}_depth_frame">
+			<sensor name="${name}/depth" type="depth">
+			    <pose> 0 0 0 0 0 0 </pose>
+			    <update_rate>30</update_rate>
+			    <camera>
+		    	    <horizontal_fov>1.518</horizontal_fov>
+				    <image>
+				        <format>R8G8B8</format>
+				        <width>848</width>
+				        <height>480</height>
+				    </image>
+				    <clip>
+				        <near>0.1</near>
+				        <far>10.0</far>
+				    </clip>
+			    </camera>
+			    <plugin name="${name}_depth_controller" filename="libgazebo_ros_camera.so">
+				    <frame_name>${name}_depth_optical_frame</frame_name>
+	                <camera_name>${name}/depth</camera_name>
+	                <ros>
+	                	<remapping>${name}/depth/depth/image_raw:=${name}/depth/image_rect_raw</remapping>
+	                	<remapping>${name}/depth/depth/camera_info:=${name}/depth/camera_info</remapping>
+	                	<remapping>${name}/depth/image_raw:=${name}/depth/color/image_raw</remapping>
+	                	<remapping>${name}/depth/camera_info:=${name}/depth/color/camera_info</remapping>
+	                	<remapping>${name}/depth/points:=${name}/depth/color/points</remapping>
+	                </ros>
 			    </plugin>
 			</sensor>
